File: src/keychain.kicad_pcb (KiCad board)
At the start: 2 copper layers, 72.8 x 101.6 mm, 9 parts, among them M1 Motor_DC, SW1 SW_Push

Commit message: add some silkscreen art
Parts:
- added G***: LOGO, LOGO, F.Cu at (96.0, 39.5)
- added G***: LOGO, LOGO, F.Cu at (123.0, 95.5)
- added G***: LOGO, LOGO, F.Cu at (150.5, 68.5)
- added G***: LOGO, LOGO, F.Cu at (146.5, 39.0)
- added G***: LOGO, LOGO, F.Cu at (97.0, 77.5)
